File: Hardware/Rev0.6rgb12Deg/trifecta.sch (KiCad schematic (older format))
At the start: 285 parts, among them J1 USB2_C_Receptacle, J2 ISP Header, SW1 RESET, SW2 Rotary_Encoder_Switch, SW3 Rotary_Encoder_Switch, SW4 Rotary_Encoder_Switch, U1 ATmega32U4-AU, U2 SRV05-4, Y1 16MHz

Commit message: 7/21
Parts:
- R7: LCSC Part# C17734 -> C269737; Mfr UNI-ROYAL(Uniroyal Elec) -> TyoHM; Part# 0805W8F5100T5E -> RMC08055105%N
Changed lines of the file:
@@
 F 1 "510Ω" V 27571 2621 50  0000 C CNN
 F 2 "Resistor_SMD:R_0805_2012Metric" H 27675 2625 50  0001 C CNN
-F 3 "https://datasheet.lcsc.com/szlcsc/Uniroyal-Elec-0805W8F5100T5E_C17734.pdf" H 27675 2625 50  0001 C CNN
-F 4 "C17734" V 27675 2625 50  0001 C CNN "LCSC Part#"
-F 5 "0805W8F5100T5E" V 27675 2625 50  0001 C CNN "Part#"
+F 3 "https://datasheet.lcsc.com/lcsc/1811101612_TyoHM-RMC08055105-N_C269737.pdf" H 27675 2625 50  0001 C CNN
+F 4 "C269737" V 27675 2625 50  0001 C CNN "LCSC Part#"
+F 5 "	RMC08055105%N" V 27675 2625 50  0001 C CNN "Part#"
 F 6 "Uniroyal Elec" V 27675 2625 50  0001 C CNN "Mrf"
-F 7 "	UNI-ROYAL(Uniroyal Elec)" H 27675 2625 50  0001 C CNN "Mfr"
+F 7 "TyoHM" H 27675 2625 50  0001 C CNN "Mfr"
 	1    27675 2625
 	0    -1   -1   0
